File: circuit/headset/headset.sch (KiCad schematic (older format))
At the start: 3 parts

Commit message: version_0.0.2
Parts:
- added J1: AudioJack3_Ground, symbol Connector:AudioJack3_Ground
- added LS1, LS2: Speaker, symbol Device:Speaker
- added MK1: Microphone, symbol Device:Microphone
- added Q3, Q4, Q5, Q6: 2SC1815, Package_TO_SOT_THT:TO-92_Inline, symbol Transistor_BJT:2SC1815
- added R1, R4: 100k, symbol Device:R_US
- added R2, R5: 1k, symbol Device:R_US
- added R3, R6, R8: 560, symbol Device:R_US
- added R7: 330, symbol Device:R_US
- added U2: LM386, symbol Amplifier_Audio:LM386
- gave numbers to parts that had none: 3
Connections:
- net at U1.2 (-): now also R1.2, R2.1
- net at U1.3 (+): now also J1.S
- net Earth: now reaches U1.4 (GND)
- net Earth: now also J1.G, MK1.1 (-), R2.2, R3.2, R5.2, R6.2, R7.2, R8.2, U2.4 (GND)
- net at Q1.3 (B), U1.5: now also R1.1
- net +5V: now reaches U1.6 (V+)
- net +5V: now also Q1.2 (C), Q2.2 (C), Q3.2 (C), Q4.2 (C), Q5.2 (C), Q6.2 (C), U2.6 (V+)
- net at Q2.1 (E): now also LS1.1, R3.1
- new net: J1.R, U2.3 (+)
- new net: J1.T, Q6.1 (E), R8.1
- new net: R4.2, R5.1, U2.2 (-)
- new net: Q3.3 (B), R4.1, U2.5
- new net: LS2.1, Q4.1 (E), R6.1
- new net: Q3.1 (E), Q4.3 (B)
- new net: MK1.2 (+), Q5.3 (B)
- new net: LS1.2, LS2.2, R7.1
- new net: Q5.1 (E), Q6.3 (B)
- no-connect marks 0 -> 6
Other:
- note added: "0.0.1"
- note added: "2021-06-16"
- note added: "Headset"
- note added: "headset"
- moved on the sheet: U1

Commit message: version_0.0.3
Parts:
- LS1, LS2: footprint (none) -> Connector_Molex:Molex_SL_171971-0002_1x02_P2.54mm_Vertical
- R1, R2, R3, R4, R5, R6, R7, R8: footprint (none) -> Resistor_THT:R_Axial_DIN0411_L9.9mm_D3.6mm_P20.32mm_Horizontal
Changed lines of the file:
@@
 F 0 "R1" V 3145 3650 50  0000 C CNN
 F 1 "100k" V 3236 3650 50  0000 C CNN
-F 2 "" V 3390 3640 50  0001 C CNN
+F 2 "Resistor_THT:R_Axial_DIN0411_L9.9mm_D3.6mm_P20.32mm_Horizontal" V 3390 3640 50  0001 C CNN
 F 3 "~" H 3350 3650 50  0001 C CNN
 	1    3350 3650
@@
 F 0 "R2" H 2918 3896 50  0000 L CNN
 F 1 "1k" H 2918 3805 50  0000 L CNN
-F 2 "" V 2890 3840 50  0001 C CNN
+F 2 "Resistor_THT:R_Axial_DIN0411_L9.9mm_D3.6mm_P20.32mm_Horizontal" V 2890 3840 50  0001 C CNN
 F 3 "~" H 2850 3850 50  0001 C CNN
 	1    2850 3850
@@
 F 0 "R3" H 4818 3796 50  0000 L CNN
 F 1 "560" H 4818 3705 50  0000 L CNN
-F 2 "" V 4790 3740 50  0001 C CNN
+F 2 "Resistor_THT:R_Axial_DIN0411_L9.9mm_D3.6mm_P20.32mm_Horizontal" V 4790 3740 50  0001 C CNN
 F 3 "~" H 4750 3750 50  0001 C CNN
 	1    4750 3750
@@
 F 0 "R4" V 6045 3650 50  0000 C CNN
 F 1 "100k" V 6136 3650 50  0000 C CNN
-F 2 "" V 6290 3640 50  0001 C CNN
+F 2 "Resistor_THT:R_Axial_DIN0411_L9.9mm_D3.6mm_P20.32mm_Horizontal" V 6290 3640 50  0001 C CNN
 F 3 "~" H 6250 3650 50  0001 C CNN
 	1    6250 3650
@@
 F 0 "R5" H 5818 3896 50  0000 L CNN
 F 1 "1k" H 5818 3805 50  0000 L CNN
-F 2 "" V 5790 3840 50  0001 C CNN
+F 2 "Resistor_THT:R_Axial_DIN0411_L9.9mm_D3.6mm_P20.32mm_Horizontal" V 5790 3840 50  0001 C CNN
 F 3 "~" H 5750 3850 50  0001 C CNN
 	1    5750 3850
@@
 F 0 "R6" H 7718 3796 50  0000 L CNN
 F 1 "560" H 7718 3705 50  0000 L CNN
-F 2 "" V 7690 3740 50  0001 C CNN
+F 2 "Resistor_THT:R_Axial_DIN0411_L9.9mm_D3.6mm_P20.32mm_Horizontal" V 7690 3740 50  0001 C CNN
 F 3 "~" H 7650 3750 50  0001 C CNN
 	1    7650 3750
@@
 F 0 "LS1" H 9720 3096 50  0000 L CNN
 F 1 "Speaker" H 9720 3005 50  0000 L CNN
-F 2 "" H 9550 2900 50  0001 C CNN
+F 2 "Connector_Molex:Molex_SL_171971-0002_1x02_P2.54mm_Vertical" H 9550 2900 50  0001 C CNN
 F 3 "~" H 9540 3050 50  0001 C CNN
 	1    9550 3100
@@
 F 0 "LS2" H 9720 3596 50  0000 L CNN
 F 1 "Speaker" H 9720 3505 50  0000 L CNN
-F 2 "" H 9550 3400 50  0001 C CNN
+F 2 "Connector_Molex:Molex_SL_171971-0002_1x02_P2.54mm_Vertical" H 9550 3400 50  0001 C CNN
 F 3 "~" H 9540 3550 50  0001 C CNN
 	1    9550 3600
@@
 F 0 "R7" H 8318 3846 50  0000 L CNN
 F 1 "330" H 8318 3755 50  0000 L CNN
-F 2 "" V 8290 3790 50  0001 C CNN
+F 2 "Resistor_THT:R_Axial_DIN0411_L9.9mm_D3.6mm_P20.32mm_Horizontal" V 8290 3790 50  0001 C CNN
 F 3 "~" H 8250 3800 50  0001 C CNN
 	1    8250 3800
@@
 F 0 "R8" H 3668 6096 50  0000 L CNN
 F 1 "560" H 3668 6005 50  0000 L CNN
-F 2 "" V 3640 6040 50  0001 C CNN
+F 2 "Resistor_THT:R_Axial_DIN0411_L9.9mm_D3.6mm_P20.32mm_Horizontal" V 3640 6040 50  0001 C CNN
 F 3 "~" H 3600 6050 50  0001 C CNN
 	1    3600 6050
